File: MAINN.kicad_pcb (KiCad board)
At the start: 2 copper layers, 19 parts, among them J1 BOOT, J2 PROG, Q1 BC847, U2 ESP_32WROOM_E, U3 MCP_RTC, Y1 32K

Commit message: Auto-commit on 2025-08-22 15:21:51
Parts:
- removed C1, C2: 22pF_0805, fevino:C_0603
- removed C3, C4, C5: .1uF, fevino:C_0603
- removed D1: ~, Diode_SMD:D_SOD-123F
- removed J1: BOOT, Connector_PinHeader_2.54mm:PinHeader_1x02_P2.54mm_Vertical
- removed J2: PROG, Connector_PinSocket_2.54mm:PinSocket_1x04_P2.54mm_Vertical
- removed K1: ~, fevino:HF32FV-G
- removed Q1: BC847, Package_TO_SOT_SMD:SOT-23
- removed R1: 1K, Resistor_SMD:R_0805_2012Metric
- removed R2, R3, R4: 4K7_0805, fevino:R_0603
- removed U1: ~, Battery:BatteryHolder_LINX_BAT-HLD-012-SMT
- removed U2: ESP_32WROOM_E, fevino:esp32-wroom-32e
- removed U3: MCP_RTC, fevino:rtc
- removed U4: ~, fevino:terminal_2pin
- removed Y1: 32K, fevino:crystal
Routing:
- net /vBat: track 13.5 -> 0.00 mm, vias 1 -> 0
- net /Net-(U3-X1): track 8.93 -> 0.00 mm
- net /Net-(U3-X2): track 5.72 -> 0.00 mm
Other:
- board text added: "MAINN_layer : B.Adhesive"
- board text added: "MAINN_layer : B.Courtyard"
- board text added: "MAINN_layer : B.Cu"
- board text added: "MAINN_layer : B.Paste"
- board text added: "MAINN_layer : B.Silkscreen"
- board text added: "MAINN_layer : Edge.Cuts"
- board text added: "MAINN_layer : F.Adhesive"
- board text added: "MAINN_layer : F.Courtyard"
- board text added: "MAINN_layer : F.Cu"
- board text added: "MAINN_layer : F.Paste"
- board text added: "MAINN_layer : F.Silkscreen"
