File: MAINN.kicad_pcb (KiCad board)
At the start: 2 copper layers, 19 parts, among them J1 BOOT, J2 PROG, Q1 BC847, U2 ESP_32WROOM_E, U3 MCP_RTC, Y1 32K

Commit message: Auto-commit on 2025-08-22 14:45:50
Parts:
- moved J2 233.5 mm to (84.8, 76.3)
- moved K1 233.5 mm to (104.0, 71.3)
- moved R1 233.5 mm to (111.0, 85.5)
- moved U4 233.5 mm to (104.0, 83.2)
- moved C3 233.5 mm to (116.2, 79.6)
- moved C4 233.5 mm to (116.2, 82.3)
- moved C5 233.5 mm to (116.2, 85.1)
- moved D1 233.5 mm to (106.0, 85.7)
- moved J1 233.5 mm to (94.2, 82.9)
- moved Q1 233.5 mm to (99.0, 83.0)
- moved R2 233.5 mm to (120.5, 73.8)
- moved R3 233.5 mm to (120.5, 76.3)
- moved R4 233.5 mm to (120.5, 78.8)
- moved U2 233.5 mm to (83.2, 73.2)
Changed lines of the file:
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@@
 	(footprint "fevino:esp32-wroom-32e"
 		(layer "F.Cu")
-		(at 316.315 59.68)
+		(at 83.165 73.205)
 		(property "Reference" "U2"
 			(at -2.58 0.93 0)
@@
 	(footprint "Connector_PinSocket_2.54mm:PinSocket_1x04_P2.54mm_Vertical"
 		(layer "F.Cu")
-		(at 317.915 62.78)
+		(at 84.765 76.305)
 		(descr "Through hole straight socket strip, 1x04, 2.54mm pitch, single row (from Kicad 4.0.7), script generated")
 		(tags "Through hole socket strip THT 1x04 2.54mm single row")
@@
 	(footprint "Resistor_SMD:R_0805_2012Metric"
 		(layer "F.Cu")
-		(at 344.125 71.94)
+		(at 110.975 85.465)
 		(descr "Resistor SMD 0805 (2012 Metric), square (rectangular) end terminal, IPC-7351 nominal, (Body size source: IPC-SM-782 page 72, https://www.pcb-3d.com/wordpress/wp-content/uploads/ipc-sm-782a_amendment_1_and_2.pdf), generated with kicad-footprint-generator")
 		(tags "resistor")
@@
 	(footprint "fevino:R_0603"
 		(layer "F.Cu")
-		(at 353.655 62.78)
+		(at 120.505 76.305)
 		(property "Reference" "R3"
 			(at 0.95 3.1 0)
@@
 	(footprint "fevino:C_0603"
 		(layer "F.Cu")
-		(at 349.395 68.82)
+		(at 116.245 82.345)
 		(property "Reference" "C4"
 			(at 0.655 -1.23 0)
@@
 	(footprint "fevino:C_0603"
 		(layer "F.Cu")
-		(at 349.395 66.06)
+		(at 116.245 79.585)
 		(property "Reference" "C3"
 			(at 0.655 -1.23 0)
@@
 	(footprint "Package_TO_SOT_SMD:SOT-23"
 		(layer "F.Cu")
-		(at 332.135 69.43)
+		(at 98.985 82.955)
 		(descr "SOT, 3 Pin (JEDEC TO-236 Var AB https://www.jedec.org/document_search?search_api_views_fulltext=TO-236), generated with kicad-footprint-generator ipc_gullwing_generator.py")
 		(tags "SOT TO_SOT_SMD")
@@
 	(footprint "fevino:C_0603"
 		(layer "F.Cu")
-		(at 349.395 71.58)
+		(at 116.245 85.105)
 		(property "Reference" "C5"
 			(at 0.655 -1.23 0)
@@
 	(footprint "fevino:R_0603"
 		(layer "F.Cu")
-		(at 353.655 65.28)
+		(at 120.505 78.805)
 		(property "Reference" "R4"
 			(at 0.95 3.1 0)
@@
 	(footprint "fevino:R_0603"
 		(layer "F.Cu")
-		(at 353.655 60.28)
+		(at 120.505 73.805)
 		(property "Reference" "R2"
 			(at 0.95 3.1 0)
@@
 	(footprint "Connector_PinHeader_2.54mm:PinHeader_1x02_P2.54mm_Vertical"
 		(layer "F.Cu")
-		(at 327.335 69.35)
+		(at 94.185 82.875)
 		(descr "Through hole straight pin header, 1x02, 2.54mm pitch, single row")
 		(tags "Through hole pin header THT 1x02 2.54mm single row")
@@
 	(footprint "fevino:terminal_2pin"
 		(layer "F.Cu")
-		(at 337.125 69.69)
+		(at 103.975 83.215)
 		(property "Reference" "U4"
 			(at 5.91 1.15 0)
@@
 	(footprint "Diode_SMD:D_SOD-123F"
 		(layer "F.Cu")
-		(at 339.145 72.14)
+		(at 105.995 85.665)
 		(descr "D_SOD-123F")
 		(tags "D_SOD-123F")
@@
 	(footprint "fevino:HF32FV-G"
 		(layer "F.Cu")
-		(at 337.125 57.78)
+		(at 103.975 71.305)
 		(property "Reference" "K1"
 			(at 9.344 -7.92 0)

Commit message: Auto commit
Parts:
- moved Y1 131.6 mm to (194.8, 32.0)
- moved U3 113.4 mm to (176.0, 33.2)
- moved U1 103.8 mm to (157.2, 33.3)
- moved U4 92.9 mm to (185.4, 38.5)
- moved U2 87.6 mm to (166.6, 46.7)
- moved C3 85.1 mm to (44.4, 33.9)
- moved C4 79.0 mm to (53.8, 33.9)
- moved C5 73.7 mm to (63.2, 33.9)
- moved D1 62.1 mm to (72.6, 33.3)
- moved R1 52.9 mm to (119.6, 33.3)
- moved R4 52.7 mm to (147.8, 33.8)
- moved J1 52.3 mm to (82.0, 32.0)
- moved Q1 50.9 mm to (110.2, 33.4)
- moved J2 47.3 mm to (91.4, 29.5)
- moved R3 46.1 mm to (138.4, 33.8)
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Routing:
- net /vBat: track 13.5 -> 28.2 mm
- net /Net-(U3-X1): track 8.93 -> 0.00 mm
- net /Net-(U3-X2): track 5.72 -> 0.00 mm
Changed lines of the file:
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@@
 	(footprint "fevino:esp32-wroom-32e"
 		(layer "F.Cu")
-		(at 83.165 73.205)
+		(at 166.608333 46.675)
 		(property "Reference" "U2"
 			(at -2.58 0.93 0)
@@
 	(footprint "Connector_PinSocket_2.54mm:PinSocket_1x04_P2.54mm_Vertical"
 		(layer "F.Cu")
-		(at 84.765 76.305)
+		(at 91.430555 29.475)
 		(descr "Through hole straight socket strip, 1x04, 2.54mm pitch, single row (from Kicad 4.0.7), script generated")
 		(tags "Through hole socket strip THT 1x04 2.54mm single row")
@@
 	(footprint "Resistor_SMD:R_0805_2012Metric"
 		(layer "F.Cu")
-		(at 110.975 85.465)
+		(at 119.622222 33.275)
 		(descr "Resistor SMD 0805 (2012 Metric), square (rectangular) end terminal, IPC-7351 nominal, (Body size source: IPC-SM-782 page 72, https://www.pcb-3d.com/wordpress/wp-content/uploads/ipc-sm-782a_amendment_1_and_2.pdf), generated with kicad-footprint-generator")
 		(tags "resistor")
@@
 	(footprint "fevino:R_0603"
 		(layer "F.Cu")
-		(at 120.505 76.305)
+		(at 138.416666 33.775)
 		(property "Reference" "R3"
 			(at 0.95 3.1 0)
@@
 	(footprint "fevino:C_0603"
 		(layer "F.Cu")
-		(at 116.245 82.345)
+		(at 53.841666 33.905)
 		(property "Reference" "C4"
 			(at 0.655 -1.23 0)
@@
 	(footprint "fevino:C_0603"
 		(layer "F.Cu")
-		(at 116.245 79.585)
+		(at 44.444444 33.905)
 		(property "Reference" "C3"
 			(at 0.655 -1.23 0)
@@
 	(footprint "Battery:BatteryHolder_LINX_BAT-HLD-012-SMT"
 		(layer "F.Cu")
-		(at 57.175 60.85 -90)
+		(at 157.211111 33.275 -90)
 		(descr "SMT battery holder for CR1216/1220/1225, https://linxtechnologies.com/wp/wp-content/uploads/bat-hld-012-smt.pdf")
 		(tags "battery holder coin cell cr1216 cr1220 cr1225")
@@
 	(footprint "Package_TO_SOT_SMD:SOT-23"
 		(layer "F.Cu")
-		(at 98.985 82.955)
+		(at 110.225 33.35)
 		(descr "SOT, 3 Pin (JEDEC TO-236 Var AB https://www.jedec.org/document_search?search_api_views_fulltext=TO-236), generated with kicad-footprint-generator ipc_gullwing_generator.py")
 		(tags "SOT TO_SOT_SMD")
@@
 	(footprint "fevino:C_0603"
 		(layer "F.Cu")
-		(at 116.245 85.105)
+		(at 63.238888 33.905)
 		(property "Reference" "C5"
 			(at 0.655 -1.23 0)
@@
 	(footprint "fevino:R_0603"
 		(layer "F.Cu")
-		(at 120.505 78.805)
+		(at 147.813888 33.775)
 		(property "Reference" "R4"
 			(at 0.95 3.1 0)
@@
 	(footprint "fevino:R_0603"
 		(layer "F.Cu")
-		(at 120.505 73.805)
+		(at 129.019444 33.775)
 		(property "Reference" "R2"
 			(at 0.95 3.1 0)
@@
 	(footprint "Connector_PinHeader_2.54mm:PinHeader_1x02_P2.54mm_Vertical"
 		(layer "F.Cu")
-		(at 94.185 82.875)
+		(at 82.033333 32)
 		(descr "Through hole straight pin header, 1x02, 2.54mm pitch, single row")
 		(tags "Through hole pin header THT 1x02 2.54mm single row")
@@
 	(footprint "fevino:crystal"
 		(layer "F.Cu")
-		(at 65.9 58.65 180)
+		(at 194.8 32.025 180)
 		(property "Reference" "Y1"
 			(at 0 -0.5 0)
@@
 	(footprint "fevino:terminal_2pin"
 		(layer "F.Cu")
-		(at 103.975 83.215)
+		(at 185.402777 38.48)
 		(property "Reference" "U4"
 			(at 5.91 1.15 0)
@@
 	(footprint "Diode_SMD:D_SOD-123F"
 		(layer "F.Cu")
-		(at 105.995 85.665)
+		(at 72.636111 33.275)
 		(descr "D_SOD-123F")
 		(tags "D_SOD-123F")
@@
 	(footprint "fevino:HF32FV-G"
 		(layer "F.Cu")
-		(at 103.975 71.305)
+		(at 100.827777 38.425)
 		(property "Reference" "K1"
 			(at 9.344 -7.92 0)
@@
 	(footprint "fevino:C_0603"
 		(layer "B.Cu")
-		(at 58.67 59.87)
+		(at 35.047222 32.645)
 		(property "Reference" "C2"
 			(at 0.655 1.23 0)
@@
 	(footprint "fevino:rtc"
 		(layer "B.Cu")
-		(at 65.92 60.305)
+		(at 176.005555 33.1725)
 		(property "Reference" "U3"
 			(at -8.2 -1 0)
@@
 	(footprint "fevino:C_0603"
 		(layer "B.Cu")
-		(at 58.795 61.53)
+		(at 25.65 32.645)
 		(property "Reference" "C1"
 			(at 0.655 1.23 0)
@@
 	)
 	(segment
-		(start 61.1 62.26)
-		(end 63.475 62.26)
+		(start 57.525 33.1)
+		(end 57.175 33.45)
 		(width 0.4)
-		(layer "B.Cu")
-		(net 2)
+		(layer "F.Cu")
+		(net 4)
 	)
 	(segment
-		(start 63.475 62.26)
-		(end 63.475 63.775)
+		(start 57.525 32.5625)
+		(end 57.525 33.9875)
 		(width 0.4)
-		(layer "B.Cu")
-		(net 2)
+		(layer "F.Cu")
+		(net 4)
+	)
+	(via
+		(at 57.525 33.275)
+		(size 0.6)
+		(drill 0.2)
+		(layers "F.Cu" "B.Cu")
+		(net 4)
 	)
 	(segment
-		(start 63.95 64.25)
-		(end 64.9 64.25)
+		(start 60.65 34.8375)
+		(end 57.525 31.7125)
 		(width 0.4)
 		(layer "B.Cu")
-		(net 2)
+		(net 4)
 	)
-	(arc
-		(start 64.9 64.25)
-		(mid 64.970711 64.220711)
-		(end 65 64.15)
+	(segment
+		(start 61.97 33.935)
+		(end 60.65 32.615)
 		(width 0.4)
 		(layer "B.Cu")
-		(net 2)
+		(net 4)
 	)
-	(arc
-		(start 63.475 63.775)
-		(mid 63.614124 64.110876)
-		(end 63.95 64.25)
+	(segment
+		(start 63.475 33.275)
+		(end 66.215 33.275)
 		(width 0.4)
 		(layer "B.Cu")
-		(net 2)
+		(net 4)
 	)
 	(segment
-		(start 63.475 60.99)
-		(end 66.215 60.99)
+		(start 66.75 32.0375)
+		(end 66.75 34.5125)
 		(width 0.4)
 		(layer "B.Cu")
-		(net 3)
+		(net 4)
 	)
 	(segment
-		(start 66.75 61.525)
-		(end 66.75 64)
+		(start 63.475 33.275)
+		(end 61.97 33.275)
 		(width 0.4)
 		(layer "B.Cu")
-		(net 3)
+		(net 4)
 	)
 	(segment
-		(start 62.036875 60.99)
-		(end 63.475 60.99)
+		(start 61.1 33.275)
+		(end 63.475 33.275)
 		(width 0.4)
 		(layer "B.Cu")
-		(net 3)
+		(net 4)
 	)
 	(segment
-		(start 61.646875 60.6)
-		(end 62.036875 60.99)
+		(start 63.475 32.5175)
+		(end 63.475 34.0325)
 		(width 0.4)
 		(layer "B.Cu")
-		(net 3)
+		(net 4)
 	)
 	(segment
-		(start 60.975 60.6)
-		(end 61.646875 60.6)
+		(start 62.036875 33.275)
+		(end 63.475 33.275)
 		(width 0.4)
 		(layer "B.Cu")
-		(net 3)
+		(net 4)
 	)
-	(arc
-		(start 66.215 60.99)
-		(mid 66.593302 61.146698)
-		(end 66.75 61.525)
+	(segment
+		(start 61.646875 33.08)
+		(end 62.036875 33.47)
 		(width 0.4)
 		(layer "B.Cu")
-		(net 3)
+		(net 4)
 	)
-	(arc
-		(start 66.75 64)
-		(mid 66.793934 64.106066)
-		(end 66.9 64.15)
+	(segment
+		(start 63.95 33.275)
+		(end 64.9 33.275)
 		(width 0.4)
 		(layer "B.Cu")
-		(net 3)
+		(net 4)
 	)
 	(segment
-		(start 57.525 52.9)
-		(end 57.175 53.25)
+		(start 60.975 33.275)
+		(end 61.646875 33.275)
 		(width 0.4)
-		(layer "F.Cu")
+		(layer "B.Cu")
 		(net 4)
 	)
 	(segment
-		(start 57.525 51.475)
-		(end 57.525 52.9)
+		(start 57.525 35.175)
+		(end 57.525 31.375)
 		(width 0.4)
-		(layer "F.Cu")
-		(net 4)
-	)
-	(via
-		(at 57.525 51.475)
-		(size 0.6)
-		(drill 0.2)
-		(layers "F.Cu" "B.Cu")
+		(layer "B.Cu")
 		(net 4)
 	)
-	(segment
-		(start 60.65 58.4)
-		(end 57.525 55.275)
+	(arc
+		(start 64.9 33.325)
+		(mid 64.970711 33.295711)
+		(end 65 33.225)
 		(width 0.4)
 		(layer "B.Cu")
 		(net 4)
 	)
-	(segment
-		(start 61.97 59.72)
-		(end 60.65 58.4)
+	(arc
+		(start 66.215 33.0075)
+		(mid 66.593302 33.164198)
+		(end 66.75 33.5425)
 		(width 0.4)
 		(layer "B.Cu")
 		(net 4)
 	)
-	(segment
-		(start 63.475 59.72)
-		(end 61.97 59.72)
+	(arc
+		(start 66.75 33.2)
+		(mid 66.793934 33.306066)
+		(end 66.9 33.35)
 		(width 0.4)
 		(layer "B.Cu")
 		(net 4)
 	)
-	(segment
-		(start 57.525 55.275)
-		(end 57.525 51.475)
+	(arc
+		(start 63.475 33.0375)
+		(mid 63.614124 33.373376)
+		(end 63.95 33.5125)
 		(width 0.4)
 		(layer "B.Cu")

Commit message: Auto commit
Routing:
- added copper zone on B.Cu, net Net-(Q1-E)
- added copper zone on F.Cu, net Net-(Q1-E)
Changed lines of the file:
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@@
 		(net 4)
+	)
+	(zone
+		(net 42)
+		(net_name "Net-(Q1-E)")
+		(layers "F.Cu" "B.Cu")
+		(name "DDE")
+		(hatch edge 0.5)
+		(connect_pads
+			(clearance 0)
+		)
+		(min_thickness 0.25)
+		(filled_areas_thickness no)
+		(fill
+			(thermal_gap 0.5)
+			(thermal_bridge_width 0.5)
+		)
+		(polygon
+			(pts
+				(xy 12.175 9.55) (xy 216.6 9.55) (xy 216.6 62) (xy 12.175 62)
+			)
+		)
 	)
 	(embedded_fonts no)

Commit message: Auto commit
Parts:
- removed C1, C2: 22pF_0805, fevino:C_0603
- removed C3, C4, C5: .1uF, fevino:C_0603
- removed D1: ~, Diode_SMD:D_SOD-123F
- removed J1: BOOT, Connector_PinHeader_2.54mm:PinHeader_1x02_P2.54mm_Vertical
- removed J2: PROG, Connector_PinSocket_2.54mm:PinSocket_1x04_P2.54mm_Vertical
- removed K1: ~, fevino:HF32FV-G
- removed Q1: BC847, Package_TO_SOT_SMD:SOT-23
- removed R1: 1K, Resistor_SMD:R_0805_2012Metric
- removed R2, R3, R4: 4K7_0805, fevino:R_0603
- removed U1: ~, Battery:BatteryHolder_LINX_BAT-HLD-012-SMT
- removed U2: ESP_32WROOM_E, fevino:esp32-wroom-32e
- removed U3: MCP_RTC, fevino:rtc
- removed U4: ~, fevino:terminal_2pin
- removed Y1: 32K, fevino:crystal
Routing:
- net /vBat: track 28.2 -> 0.00 mm, vias 1 -> 0
- removed copper zone on B.Cu, net Net-(Q1-E)
- removed copper zone on F.Cu, net Net-(Q1-E)
Other:
- board text added: "MAINN_layer : B.Adhesive"
- board text added: "MAINN_layer : B.Courtyard"
- board text added: "MAINN_layer : B.Cu"
- board text added: "MAINN_layer : B.Paste"
- board text added: "MAINN_layer : B.Silkscreen"
- board text added: "MAINN_layer : Edge.Cuts"
- board text added: "MAINN_layer : F.Adhesive"
- board text added: "MAINN_layer : F.Courtyard"
- board text added: "MAINN_layer : F.Cu"
- board text added: "MAINN_layer : F.Paste"
- board text added: "MAINN_layer : F.Silkscreen"
