File: MAINN.kicad_sch (KiCad schematic)
At the start: 19 parts, among them J1 BOOT, J2 PROG, Q1 BC847, U2 ESP_32WROOM_E, U3 MCP_RTC, Y1 32K

Commit message: Auto-commit on 2025-08-22 15:21:51
Parts:
- removed C1, C2: 22pF_0805, fevino:C_0603, symbol Device:C
- removed C3, C4, C5: .1uF, fevino:C_0603, symbol Device:C
- removed D1: ~, Diode_SMD:D_SOD-123F, symbol fevino:1N4148_SOD
- removed J1: BOOT, Connector_PinHeader_2.54mm:PinHeader_1x02_P2.54mm_Vertical, symbol Connector_Generic:Conn_01x02
- removed J2: PROG, Connector_PinSocket_2.54mm:PinSocket_1x04_P2.54mm_Vertical, symbol Connector_Generic:Conn_01x04
- removed K1: ~, fevino:HF32FV-G, symbol fevino:HF32FV-G
- removed Q1: BC847, Package_TO_SOT_SMD:SOT-23, symbol Transistor_BJT:BC847
- removed R1: 1K, Resistor_SMD:R_0805_2012Metric, symbol Device:R
- removed R2, R3, R4: 4K7_0805, fevino:R_0603, symbol Device:R
- removed U1: ~, Battery:BatteryHolder_LINX_BAT-HLD-012-SMT, symbol fevino:battery
- removed U2: ESP_32WROOM_E, fevino:esp32-wroom-32e, symbol fevino:esp32-wroom-32e
- removed U3: MCP_RTC, fevino:rtc, symbol fevino:rtc
- removed U4: ~, fevino:terminal_2pin, symbol fevino:terminal_2pin
- removed Y1: 32K, fevino:crystal, symbol Device:Crystal
- added J1: Screw_Terminal_2_P5.00mm, TerminalBlock_Phoenix:TerminalBlock_Phoenix_PT-1,5-2-5.0-H_1x02_P5.00mm_Horizontal, symbol PCM_SL_Screw_Terminal:Screw_Terminal_2_P5.00mm
- added U1: 2 pin terminal 5.08mm XYU 128 2 pin, fevino:terminal_2pin, symbol fevino:terminal_2pin
Other:
- note removed: "ESP"
- note removed: "RTC"

Commit message: Auto commit
Parts:
- removed J1: Screw_Terminal_2_P5.00mm, TerminalBlock_Phoenix:TerminalBlock_Phoenix_PT-1,5-2-5.0-H_1x02_P5.00mm_Horizontal, symbol PCM_SL_Screw_Terminal:Screw_Terminal_2_P5.00mm
Changed lines of the file:
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@@
-		)
-	)
-	(symbol
-		(lib_id "PCM_SL_Screw_Terminal:Screw_Terminal_2_P5.00mm")
-		(at 156.21 62.23 0)
-		(unit 1)
-		(exclude_from_sim no)
-		(in_bom yes)
-		(on_board yes)
-		(dnp no)
-		(fields_autoplaced yes)
-		(property "Reference" "J1"
-			(at 160.02 60.9599 0)
-			(effects
-				(font
-					(size 1.27 1.27)
-				)
-				(justify left)
-			)
-		)
-		(property "Value" "Screw_Terminal_2_P5.00mm"
-			(at 160.02 63.4999 0)
-			(effects
-				(font
-					(size 1.27 1.27)
-				)
-				(justify left)
-			)
-		)
-		(property "Footprint" "TerminalBlock_Phoenix:TerminalBlock_Phoenix_PT-1,5-2-5.0-H_1x02_P5.00mm_Horizontal"
-			(at 157.48 68.58 0)
-			(effects
-				(font
-					(size 1.27 1.27)
-				)
-				(hide yes)
-			)
-		)
-		(property "Datasheet" ""
-			(at 156.21 62.23 0)
-			(effects
-				(font
-					(size 1.27 1.27)
-				)
-				(hide yes)
-			)
-		)
-		(property "Description" ""
-			(at 156.21 62.23 0)
-			(effects
-				(font
-					(size 1.27 1.27)
-				)
-				(hide yes)
-			)
-		)
-		(pin "1"
-		)
-		(pin "2"
-		)
-		(instances
-			(project ""
-				(path "/8469cd9a-15fe-4677-a617-64af849f0980"
-					(reference "J1")
-					(unit 1)
-				)
-			)
 		)
 	)
